File: tsuka60.sch (KiCad schematic (older format))
At the start: 14 parts

Commit message: basic matrix layout complete
Parts:
- added D? (x75): D_Small, symbol Device:D_Small
- added MX? (x75): MX-LED, symbol MX_Alps_Hybrid:MX-LED
Connections:
- net Row1: now reaches U?.1 (PE6)
- net Row1: now also D?.1 (K), D?.1 (K), D?.1 (K), D?.1 (K), D?.1 (K), D?.1 (K), D?.1 (K), D?.1 (K), D?.1 (K), D?.1 (K), D?.1 (K), D?.1 (K), D?.1 (K), D?.1 (K), D?.1 (K)
- net Col14: now reaches U?.18 (PD0)
- net Col14: now also MX?.1 (COL), MX?.1 (COL), MX?.1 (COL), MX?.1 (COL), MX?.1 (COL)
- net Col13: now reaches U?.19 (PD1)
- net Col13: now also MX?.1 (COL), MX?.1 (COL), MX?.1 (COL), MX?.1 (COL), MX?.1 (COL)
- net Col12: now reaches U?.20 (PD2)
- net Col12: now also MX?.1 (COL), MX?.1 (COL), MX?.1 (COL), MX?.1 (COL), MX?.1 (COL)
- net Col11: now reaches U?.21 (PD3)
- net Col11: now also MX?.1 (COL), MX?.1 (COL), MX?.1 (COL), MX?.1 (COL), MX?.1 (COL)
- net Row2: now reaches U?.22 (PD5)
- net Row2: now also D?.1 (K), D?.1 (K), D?.1 (K), D?.1 (K), D?.1 (K), D?.1 (K), D?.1 (K), D?.1 (K), D?.1 (K), D?.1 (K), D?.1 (K), D?.1 (K), D?.1 (K), D?.1 (K), D?.1 (K)
- net Col10: now reaches U?.25 (PD4)
- net Col10: now also MX?.1 (COL), MX?.1 (COL), MX?.1 (COL), MX?.1 (COL), MX?.1 (COL)
- net Col9: now reaches U?.26 (PD6)
- net Col9: now also MX?.1 (COL), MX?.1 (COL), MX?.1 (COL), MX?.1 (COL), MX?.1 (COL)
- net Row3: now reaches U?.28 (PB4)
- net Row3: now also D?.1 (K), D?.1 (K), D?.1 (K), D?.1 (K), D?.1 (K), D?.1 (K), D?.1 (K), D?.1 (K), D?.1 (K), D?.1 (K), D?.1 (K), D?.1 (K), D?.1 (K), D?.1 (K), D?.1 (K)
- net Row4: now reaches U?.29 (PB5)
- net Row4: now also D?.1 (K), D?.1 (K), D?.1 (K), D?.1 (K), D?.1 (K), D?.1 (K), D?.1 (K), D?.1 (K), D?.1 (K), D?.1 (K), D?.1 (K), D?.1 (K), D?.1 (K), D?.1 (K), D?.1 (K)
- net Col8: now reaches U?.30 (PB6)
- net Col8: now also MX?.1 (COL), MX?.1 (COL), MX?.1 (COL), MX?.1 (COL), MX?.1 (COL)
- net Col7: now reaches U?.31 (PC6)
- net Col7: now also MX?.1 (COL), MX?.1 (COL), MX?.1 (COL), MX?.1 (COL), MX?.1 (COL)
- net Col6: now reaches U?.32 (PC7)
- net Col6: now also MX?.1 (COL), MX?.1 (COL), MX?.1 (COL), MX?.1 (COL), MX?.1 (COL)
- net Col5: now reaches U?.36 (PF7)
- net Col5: now also MX?.1 (COL), MX?.1 (COL), MX?.1 (COL), MX?.1 (COL), MX?.1 (COL)
- net Col4: now reaches U?.37 (PF6)
- net Col4: now also MX?.1 (COL), MX?.1 (COL), MX?.1 (COL), MX?.1 (COL), MX?.1 (COL)
- net Col3: now reaches U?.38 (PF5)
- net Col3: now also MX?.1 (COL), MX?.1 (COL), MX?.1 (COL), MX?.1 (COL), MX?.1 (COL)
- net Col2: now reaches U?.39 (PF4)
- net Col2: now also MX?.1 (COL), MX?.1 (COL), MX?.1 (COL), MX?.1 (COL), MX?.1 (COL)
- net Col1: now reaches U?.40 (PF1)
- net Col1: now also MX?.1 (COL), MX?.1 (COL), MX?.1 (COL), MX?.1 (COL), MX?.1 (COL)
- net Col0: now reaches U?.41 (PF0)
- net Col0: now also MX?.1 (COL), MX?.1 (COL), MX?.1 (COL), MX?.1 (COL), MX?.1 (COL)
- net Row0: now reaches U?.8 (PB0)
- net Row0: now also D?.1 (K), D?.1 (K), D?.1 (K), D?.1 (K), D?.1 (K), D?.1 (K), D?.1 (K), D?.1 (K), D?.1 (K), D?.1 (K), D?.1 (K), D?.1 (K), D?.1 (K), D?.1 (K), D?.1 (K)
- new net: D?.2 (A), MX?.2 (ROW) (x75)
Other:
- moved on the sheet: C?, F?, R?, SW?, U?, USB?, Y?

Commit message: assigned footprints and generated netlist
Parts:
- removed MX? (x60): MX-LED, symbol MX_Alps_Hybrid:MX-LED
- added MX16, MX17, MX18, MX19, MX20, MX21, MX22, MX23, MX24, MX25, MX26, MX27, MX28, MX29, MX30, MX31, MX32, MX33, MX34, MX35, MX36, MX37, MX38, MX39, MX40, MX41, MX42, MX43, MX44, MX45, MX46, MX47, MX48, MX49, MX50, MX51, MX52, MX53, MX54, MX55, MX56, MX57, MX58, MX59, MX60, MX61, MX62, MX63, MX64, MX65, MX66, MX67, MX68, MX69, MX70, MX71, MX72, MX73, MX74, MX75: MX-LED, MX_Alps_Hybrid:MX-1U-NoLED, symbol MX_Alps_Hybrid:MX-NoLED
- C1, C2, C3, C4, C5: renamed from C?; footprint (none) -> Capacitor_SMD:C_0805_2012Metric
- D1, D10, D11, D12, D13, D14, D15, D16, D17, D18, D19, D2, D20, D21, D22, D23, D24, D25, D26, D27, D28, D29, D3, D30, D31, D32, D33, D34, D35, D36, D37, D38, D39, D4, D40, D41, D42, D43, D44, D45, D46, D47, D48, D49, D5, D50, D51, D52, D53, D54, D55, D56, D57, D58, D59, D6, D60, D61, D62, D63, D64, D65, D66, D67, D68, D69, D7, D70, D71, D72, D73, D74, D75, D8, D9: renamed from D?; footprint (none) -> Diode_SMD:D_0805_2012Metric
- F1: renamed from F?; footprint (none) -> Fuse:Fuse_1206_3216Metric
- MX1, MX10, MX11, MX12, MX13, MX14, MX15, MX2, MX3, MX4, MX5, MX6, MX7, MX8, MX9: renamed from MX?; footprint (none) -> MX_Alps_Hybrid:MX-1U-NoLED; symbol MX_Alps_Hybrid:MX-LED -> MX_Alps_Hybrid:MX-NoLED
- R1, R2, R3, R4: renamed from R?; footprint (none) -> Resistor_SMD:R_0805_2012Metric
- SW1: renamed from SW?; footprint (none) -> random-keyboard-parts:SKQG-1155865
- USB1: renamed from USB?; footprint (none) -> random-keyboard-parts:Molex-0548190589
- Y1: renamed from Y?; footprint (none) -> Crystal:Resonator_SMD_muRata_CSTxExxV-3Pin_3.0x1.1mm
- gave numbers to parts that had none: 1
Connections:
- net Col0: now also MX46.1 (COL), MX61.1 (COL)
- net Col1: now also MX47.1 (COL), MX62.1 (COL)
- net Col10: now also MX56.1 (COL), MX71.1 (COL)
- net Col11: now also MX57.1 (COL), MX72.1 (COL)
- net Col12: now also MX58.1 (COL), MX73.1 (COL)
- net Col13: now also MX59.1 (COL), MX74.1 (COL)
- net Col14: now also MX60.1 (COL), MX75.1 (COL)
- net Col2: now also MX48.1 (COL), MX63.1 (COL)
- net Col3: now also MX49.1 (COL), MX64.1 (COL)
- net Col4: now also MX50.1 (COL), MX65.1 (COL)
- net Col5: now also MX51.1 (COL), MX66.1 (COL)
- net Col6: now also MX52.1 (COL), MX67.1 (COL)
- net Col7: now also MX53.1 (COL), MX68.1 (COL)
- net Col8: now also MX54.1 (COL), MX69.1 (COL)
- net Col9: now also MX55.1 (COL), MX70.1 (COL)
- net at D16.2 (A): now also MX16.2 (ROW)
- net at D17.2 (A): now also MX17.2 (ROW)
- net at D18.2 (A): now also MX18.2 (ROW)
- net at D19.2 (A): now also MX19.2 (ROW)
- net at D20.2 (A): now also MX20.2 (ROW)
- net at D21.2 (A): now also MX21.2 (ROW)
- net at D22.2 (A): now also MX22.2 (ROW)
- net at D23.2 (A): now also MX23.2 (ROW)
- net at D24.2 (A): now also MX24.2 (ROW)
- net at D25.2 (A): now also MX25.2 (ROW)
- net at D26.2 (A): now also MX26.2 (ROW)
- net at D27.2 (A): now also MX27.2 (ROW)
- net at D28.2 (A): now also MX28.2 (ROW)
- net at D29.2 (A): now also MX29.2 (ROW)
- net at D30.2 (A): now also MX30.2 (ROW)
- net at D31.2 (A): now also MX31.2 (ROW)
- net at D32.2 (A): now also MX32.2 (ROW)
- net at D33.2 (A): now also MX33.2 (ROW)
- net at D34.2 (A): now also MX34.2 (ROW)
- net at D35.2 (A): now also MX35.2 (ROW)
- net at D36.2 (A): now also MX36.2 (ROW)
- net at D37.2 (A): now also MX37.2 (ROW)
- net at D38.2 (A): now also MX38.2 (ROW)
- net at D39.2 (A): now also MX39.2 (ROW)
- net at D40.2 (A): now also MX40.2 (ROW)
- net at D41.2 (A): now also MX41.2 (ROW)
- net at D42.2 (A): now also MX42.2 (ROW)
- net at D43.2 (A): now also MX43.2 (ROW)
- net at D44.2 (A): now also MX44.2 (ROW)
- net at D45.2 (A): now also MX45.2 (ROW)
- net at D46.2 (A): now also MX46.2 (ROW)
- net at D47.2 (A): now also MX47.2 (ROW)
- net at D48.2 (A): now also MX48.2 (ROW)
- net at D49.2 (A): now also MX49.2 (ROW)
- net at D50.2 (A): now also MX50.2 (ROW)
- net at D51.2 (A): now also MX51.2 (ROW)
- net at D52.2 (A): now also MX52.2 (ROW)
- net at D53.2 (A): now also MX53.2 (ROW)
- net at D54.2 (A): now also MX54.2 (ROW)
- net at D55.2 (A): now also MX55.2 (ROW)
- net at D56.2 (A): now also MX56.2 (ROW)
- net at D57.2 (A): now also MX57.2 (ROW)
- net at D58.2 (A): now also MX58.2 (ROW)
- net at D59.2 (A): now also MX59.2 (ROW)
- net at D60.2 (A): now also MX60.2 (ROW)
- net at D61.2 (A): now also MX61.2 (ROW)
- net at D62.2 (A): now also MX62.2 (ROW)
- net at D63.2 (A): now also MX63.2 (ROW)
- net at D64.2 (A): now also MX64.2 (ROW)
- net at D65.2 (A): now also MX65.2 (ROW)
- net at D66.2 (A): now also MX66.2 (ROW)
- net at D67.2 (A): now also MX67.2 (ROW)
- net at D68.2 (A): now also MX68.2 (ROW)
- net at D69.2 (A): now also MX69.2 (ROW)
- net at D70.2 (A): now also MX70.2 (ROW)
- net at D71.2 (A): now also MX71.2 (ROW)
- net at D72.2 (A): now also MX72.2 (ROW)
- net at D73.2 (A): now also MX73.2 (ROW)
- net at D74.2 (A): now also MX74.2 (ROW)
- net at D75.2 (A): now also MX75.2 (ROW)

Commit message: Started component layout
Parts:
- MX31, MX45: footprint MX_Alps_Hybrid:MX-1U-NoLED -> MX_Alps_Hybrid:MX-1.75U-NoLED
- MX38, MX46, MX60: footprint MX_Alps_Hybrid:MX-1U-NoLED -> MX_Alps_Hybrid:MX-1.5U-NoLED
- MX53: footprint MX_Alps_Hybrid:MX-1U-NoLED -> MX_Alps_Hybrid:MX-2U-NoLED
Changed lines of the file:
@@
 F 0 "MX31" H 2682 4874 60  0000 C CNN
 F 1 "MX-LED" H 2682 4800 20  0000 C CNN
-F 2 "MX_Alps_Hybrid:MX-1U-NoLED" H 1975 4625 60  0001 C CNN
+F 2 "MX_Alps_Hybrid:MX-1.75U-NoLED" H 1975 4625 60  0001 C CNN
 F 3 "" H 1975 4625 60  0001 C CNN
 	1    2600 4650
@@
 F 0 "MX38" H 11432 4874 60  0000 C CNN
 F 1 "MX-LED" H 11432 4800 20  0000 C CNN
-F 2 "MX_Alps_Hybrid:MX-1U-NoLED" H 10725 4625 60  0001 C CNN
+F 2 "MX_Alps_Hybrid:MX-1.5U-NoLED" H 10725 4625 60  0001 C CNN
 F 3 "" H 10725 4625 60  0001 C CNN
 	1    11350 4650
@@
 F 0 "MX45" H 20182 4874 60  0000 C CNN
 F 1 "MX-LED" H 20182 4800 20  0000 C CNN
-F 2 "MX_Alps_Hybrid:MX-1U-NoLED" H 19475 4625 60  0001 C CNN
+F 2 "MX_Alps_Hybrid:MX-1.75U-NoLED" H 19475 4625 60  0001 C CNN
 F 3 "" H 19475 4625 60  0001 C CNN
 	1    20100 4650
@@
 F 0 "MX46" H 2682 6124 60  0000 C CNN
 F 1 "MX-LED" H 2682 6050 20  0000 C CNN
-F 2 "MX_Alps_Hybrid:MX-1U-NoLED" H 1975 5875 60  0001 C CNN
+F 2 "MX_Alps_Hybrid:MX-1.5U-NoLED" H 1975 5875 60  0001 C CNN
 F 3 "" H 1975 5875 60  0001 C CNN
 	1    2600 5900
@@
 F 0 "MX53" H 11432 6124 60  0000 C CNN
 F 1 "MX-LED" H 11432 6050 20  0000 C CNN
-F 2 "MX_Alps_Hybrid:MX-1U-NoLED" H 10725 5875 60  0001 C CNN
+F 2 "MX_Alps_Hybrid:MX-2U-NoLED" H 10725 5875 60  0001 C CNN
 F 3 "" H 10725 5875 60  0001 C CNN
 	1    11350 5900
@@
 F 0 "MX60" H 20182 6124 60  0000 C CNN
 F 1 "MX-LED" H 20182 6050 20  0000 C CNN
-F 2 "MX_Alps_Hybrid:MX-1U-NoLED" H 19475 5875 60  0001 C CNN
+F 2 "MX_Alps_Hybrid:MX-1.5U-NoLED" H 19475 5875 60  0001 C CNN
 F 3 "" H 19475 5875 60  0001 C CNN
 	1    20100 5900

Commit message: Started organising bottom rows
Parts:
- removed D37, D39, D52, D54, D66: D_Small, Diode_SMD:D_0805_2012Metric, symbol Device:D_Small
- removed MX37, MX39, MX52, MX54, MX64, MX65, MX66: MX-LED, MX_Alps_Hybrid:MX-1U-NoLED, symbol MX_Alps_Hybrid:MX-NoLED
- added MX61-1: L-CTRL, MX_Alps_Hybrid:MX-1.25U-NoLED, symbol MX_Alps_Hybrid:MX-NoLED
- added MX62-1: L-WIN, MX_Alps_Hybrid:MX-1.25U-NoLED, symbol MX_Alps_Hybrid:MX-NoLED
- added MX63-1: L-ALT, MX_Alps_Hybrid:MX-1.25U-NoLED, symbol MX_Alps_Hybrid:MX-NoLED
- added MX64-1: BACK SPACE, MX_Alps_Hybrid:MX-2.75U-ReversedStabilizers-NoLED, symbol MX_Alps_Hybrid:MX-NoLED
- added MX64-2: BACK SPACE, MX_Alps_Hybrid:MX-3U-ReversedStabilizers-NoLED, symbol MX_Alps_Hybrid:MX-NoLED
- added MX65-1: RETURN, MX_Alps_Hybrid:MX-2U-ReversedStabilizers-NoLED, symbol MX_Alps_Hybrid:MX-NoLED
- added MX65-2: RETURN, MX_Alps_Hybrid:MX-1.5U-NoLED, symbol MX_Alps_Hybrid:MX-NoLED
- added MX67-1: SPACE, MX_Alps_Hybrid:MX-2.75U-ReversedStabilizers-NoLED, symbol MX_Alps_Hybrid:MX-NoLED
- added MX67-2: SPACE, MX_Alps_Hybrid:MX-3U-ReversedStabilizers-NoLED, symbol MX_Alps_Hybrid:MX-NoLED
- added MX67-3: SPACE, MX_Alps_Hybrid:MX-6.25U-ReversedStabilizers-NoLED, symbol MX_Alps_Hybrid:MX-NoLED
- added MX69-1: R-ALT, MX_Alps_Hybrid:MX-1.25U-NoLED, symbol MX_Alps_Hybrid:MX-NoLED
- added MX70-1: R-WIN, MX_Alps_Hybrid:MX-1.25U-NoLED, symbol MX_Alps_Hybrid:MX-NoLED
- added MX71-1: R-CTRL, MX_Alps_Hybrid:MX-1.25U-NoLED, symbol MX_Alps_Hybrid:MX-NoLED
- MX61: value MX-LED -> L-CTRL; footprint MX_Alps_Hybrid:MX-1U-NoLED -> MX_Alps_Hybrid:MX-1.5U-NoLED
- MX62: value MX-LED -> L-WIN
- MX63: value MX-LED -> L-ALT; footprint MX_Alps_Hybrid:MX-1U-NoLED -> MX_Alps_Hybrid:MX-1.5U-NoLED
- MX67: value MX-LED -> SPACE; footprint MX_Alps_Hybrid:MX-1U-NoLED -> MX_Alps_Hybrid:MX-7U-NoLED
- MX68-3: renamed from MX68; value MX-LED -> LEGACY; footprint MX_Alps_Hybrid:MX-1U-NoLED -> MX_Alps_Hybrid:MX-1.25U-NoLED
- MX69: value MX-LED -> R-ALT; footprint MX_Alps_Hybrid:MX-1U-NoLED -> MX_Alps_Hybrid:MX-1.5U-NoLED
- MX70: value MX-LED -> R-WIN
- MX71: value MX-LED -> R-CTRL; footprint MX_Alps_Hybrid:MX-1U-NoLED -> MX_Alps_Hybrid:MX-1.5U-NoLED
- MX72: value MX-LED -> LEFT
- MX73: value MX-LED -> DOWN
- MX74: value MX-LED -> UP
- MX75: value MX-LED -> RIGHT
Connections:
- net Col0: now also MX61-1.1 (COL)
- net Col1: now also MX62-1.1 (COL)
- net Col10: now also MX71-1.1 (COL)
- net Col2: now also MX63-1.1 (COL)
- net Col3: now also MX64-1.1 (COL), MX64-2.1 (COL)
- net Col4: now also MX65-1.1 (COL), MX65-2.1 (COL)
- net Col6: now also MX67-1.1 (COL), MX67-2.1 (COL), MX67-3.1 (COL)
- net Col8: now also MX69-1.1 (COL)
- net Col9: now also MX70-1.1 (COL)
- net Row4: no longer D64.1 (K), D65.1 (K), D70.1 (K), D71.1 (K), D72.1 (K)
- net at D61.2 (A), MX61.2 (ROW): now also MX61-1.2 (ROW)
- net at D62.2 (A), MX62.2 (ROW): now also MX62-1.2 (ROW)
- net at D63.2 (A), MX63.2 (ROW): now also MX63-1.2 (ROW)
- net at D64.2 (A): now also MX64-1.2 (ROW), MX64-2.2 (ROW)
- net at D65.2 (A): now also MX65-1.2 (ROW), MX65-2.2 (ROW)
- net at D67.2 (A), MX67.2 (ROW): now also MX67-1.2 (ROW), MX67-2.2 (ROW), MX67-3.2 (ROW)
- net at D69.2 (A), MX69.2 (ROW): now also MX69-1.2 (ROW)
- net at D70.2 (A), MX70.2 (ROW): now also MX70-1.2 (ROW)
- net at D71.2 (A), MX71.2 (ROW): now also MX71-1.2 (ROW)

Commit message: Start with the layout of diodes
Parts:
- USB1: footprint random-keyboard-parts:Molex-0548190589 -> random-keyboard-parts:Molex-0548190519
Changed lines of the file:
@@
 F 0 "USB1" V 8287 10467 60  0000 C CNN
 F 1 "Molex-0548190589" V 8181 10467 60  0000 C CNN
-F 2 "random-keyboard-parts:Molex-0548190589" H 7750 10500 60  0001 C CNN
+F 2 "random-keyboard-parts:Molex-0548190519" H 7750 10500 60  0001 C CNN
 F 3 "" H 7750 10500 60  0001 C CNN
 	1    7750 10500

Commit message: ready for tracing
Parts:
- MX53: footprint MX_Alps_Hybrid:MX-2U-NoLED -> MX_Alps_Hybrid:MX-2U-ReversedStabilizers-NoLED
Changed lines of the file:
@@
 F 0 "MX53" H 11432 6124 60  0000 C CNN
 F 1 "MX-LED" H 11432 6050 20  0000 C CNN
-F 2 "MX_Alps_Hybrid:MX-2U-NoLED" H 10725 5875 60  0001 C CNN
+F 2 "MX_Alps_Hybrid:MX-2U-ReversedStabilizers-NoLED" H 10725 5875 60  0001 C CNN
 F 3 "" H 10725 5875 60  0001 C CNN
 	1    11350 5900

Commit message: started tracing
Connections:
- net Col0: now also MX16.1 (COL), MX31.1 (COL)
- net Col1: now also MX17.1 (COL), MX32.1 (COL)
- net Col10: now also MX26.1 (COL), MX41.1 (COL)
- net Col11: now also MX27.1 (COL), MX42.1 (COL)
- net Col12: now also MX28.1 (COL), MX43.1 (COL)
- net Col13: now also MX29.1 (COL), MX44.1 (COL)
- net Col14: now also MX30.1 (COL), MX45.1 (COL)
- net Col2: now also MX18.1 (COL), MX33.1 (COL)
- net Col3: now also MX19.1 (COL), MX34.1 (COL)
- net Col4: now also MX20.1 (COL), MX35.1 (COL)
- net Col5: now also MX21.1 (COL), MX36.1 (COL)
- net Col6: now also MX22.1 (COL)
- net Col7: now also MX23.1 (COL), MX38.1 (COL)
- net Col8: now also MX24.1 (COL)
- net Col9: now also MX25.1 (COL), MX40.1 (COL)
Changed lines of the file:
@@
 	17750 2100 17750 1250
 Wire Wire Line
-	16500 2100 16500 1250
-Wire Wire Line
 	15250 2100 15250 1250
 Wire Wire Line
@@
 	7750 1250 7750 2100
 Wire Wire Line
-	6500 2100 6500 5850
-Wire Wire Line
-	5250 2100 5250 5850
-Wire Wire Line
-	4000 2100 4000 5850
-Wire Wire Line
-	2750 2100 2750 5850
-Wire Wire Line
-	20250 2100 20250 5850
-Wire Wire Line
-	19000 2100 19000 5850
-Wire Wire Line
-	17750 2100 17750 5850
-Wire Wire Line
-	16500 2100 16500 5850
-Wire Wire Line
-	15250 2100 15250 5850
-Wire Wire Line
-	14000 2100 14000 5850
-Wire Wire Line
-	11500 2100 11500 5850
-Wire Wire Line
-	9000 2100 9000 5850
-Wire Wire Line
-	7750 2100 7750 5850
+	6500 2100 6500 3350
+Wire Wire Line
+	5250 2100 5250 3350
+Wire Wire Line
+	4000 2100 4000 3350
+Wire Wire Line
+	2750 2100 2750 3350
+Wire Wire Line
+	15250 2100 15250 3350
+Wire Wire Line
+	14000 2100 14000 3350
+Wire Wire Line
+	9000 2100 9000 3350
+Wire Wire Line
+	7750 2100 7750 3350
 Wire Wire Line
 	8650 5000 11150 5000
@@
 	11150 6250 13650 6250
 Wire Wire Line
-	12750 2100 12750 6550
+	12750 2100 12750 3350
 Wire Wire Line
 	8650 6250 11150 6250
@@
 	9050 7300 9550 7300
 Wire Wire Line
-	10250 2100 10250 6750
+	10250 2100 10250 3350
 Wire Wire Line
 	9750 7100 9925 7100
@@
 	13650 6750 13650 7300
 Connection ~ 13650 7300
+Wire Wire Line
+	19000 2100 19000 3350
+Connection ~ 19000 3350
+Wire Wire Line
+	19000 3350 19000 4600
+Connection ~ 19000 4600
+Wire Wire Line
+	19000 4600 19000 5850
+Connection ~ 17750 4600
+Wire Wire Line
+	17750 4600 17750 5850
+Wire Wire Line
+	17750 2100 17750 3350
+Wire Wire Line
+	20250 2100 20250 3350
+Connection ~ 20250 4600
+Wire Wire Line
+	20250 4600 20250 5850
+Connection ~ 20250 2100
+Connection ~ 20250 3350
+Wire Wire Line
+	20250 3350 20250 4600
+Connection ~ 20250 5850
+Connection ~ 19000 5850
+Connection ~ 17750 5850
+Wire Wire Line
+	17750 3350 17750 4600
+Connection ~ 17750 3350
+Wire Wire Line
+	16500 2100 16500 3350
+Connection ~ 16500 3350
+Wire Wire Line
+	16500 3350 16500 4600
+Connection ~ 16500 4600
+Wire Wire Line
+	16500 4600 16500 5850
+Connection ~ 15250 2100
+Connection ~ 15250 3350
+Wire Wire Line
+	15250 3350 15250 4600
+Connection ~ 14000 3350
+Wire Wire Line
+	14000 3350 14000 4600
+Connection ~ 14000 2100
+Connection ~ 12750 2100
+Connection ~ 12750 3350
+Wire Wire Line
+	12750 3350 12750 6550
+Wire Wire Line
+	11500 2100 11500 3350
+Connection ~ 11500 3350
+Wire Wire Line
+	11500 3350 11500 4600
+Connection ~ 11500 2100
+Connection ~ 10250 2100
+Connection ~ 10250 3350
+Wire Wire Line
+	10250 3350 10250 6750
+Wire Wire Line
+	11500 4600 11500 5850
+Connection ~ 11500 4600
+Connection ~ 11500 5850
+Wire Wire Line
+	14000 4600 14000 5850
+Connection ~ 14000 4600
+Wire Wire Line
+	15250 4600 15250 5850
+Connection ~ 15250 4600
+Connection ~ 9000 2100
+Connection ~ 9000 4600
+Wire Wire Line
+	9000 4600 9000 5850
+Connection ~ 9000 3350
+Wire Wire Line
+	9000 3350 9000 4600
+Connection ~ 7750 2100
+Connection ~ 7750 3350
+Wire Wire Line
+	7750 3350 7750 4600
+Connection ~ 7750 4600
+Wire Wire Line
+	7750 4600 7750 5850
+Connection ~ 6500 2100
+Connection ~ 6500 4600
+Wire Wire Line
+	6500 4600 6500 5850
+Connection ~ 6500 3350
+Wire Wire Line
+	6500 3350 6500 4600
+Connection ~ 5250 5850
+Connection ~ 5250 2100
+Connection ~ 5250 3350
+Wire Wire Line
+	5250 3350 5250 4600
+Connection ~ 5250 4600
+Wire Wire Line
+	5250 4600 5250 5850
+Connection ~ 4000 2100
+Connection ~ 4000 5850
+Connection ~ 4000 3350
+Wire Wire Line
+	4000 3350 4000 4600
+Connection ~ 4000 4600
+Wire Wire Line
+	4000 4600 4000 5850
+Connection ~ 2750 5850
+Connection ~ 2750 2100
+Connection ~ 2750 3350
+Wire Wire Line
+	2750 3350 2750 4600
+Connection ~ 2750 4600
+Wire Wire Line
+	2750 4600 2750 5850
+Connection ~ 19000 2100
+Connection ~ 17750 2100
+Wire Wire Line
+	16500 1250 16500 2100
+Connection ~ 16500 2100
 $EndSCHEMATC

Commit message: more tracing
Connections:
- net Col3: now also U1.32 (PC7); no longer U1.38 (PF5)
- net Col4: now also U1.31 (PC6); no longer U1.37 (PF6)
- net Col6: now also U1.38 (PF5); no longer U1.32 (PC7)
- net Col7: now also U1.37 (PF6); no longer U1.31 (PC6)
Changed lines of the file:
@@
 Text GLabel 5750 12950 2    50   Input ~ 0
 Col2
-Text GLabel 5750 13050 2    50   Input ~ 0
+Text GLabel 5750 11350 2    50   Input ~ 0
 Col3
-Text GLabel 5750 13150 2    50   Input ~ 0
+Text GLabel 5750 11250 2    50   Input ~ 0
 Col4
 Text GLabel 5750 13250 2    50   Input ~ 0
 Col5
-Text GLabel 5750 11350 2    50   Input ~ 0
+Text GLabel 5750 13050 2    50   Input ~ 0
 Col6
-Text GLabel 5750 11250 2    50   Input ~ 0
+Text GLabel 5750 13150 2    50   Input ~ 0
 Col7
 Text GLabel 5750 10950 2    50   Input ~ 0
