File: tsuka60.sch (KiCad schematic (older format))
At the start: 172 parts, among them SW1 SW_Push, U1 ATmega32U4-AU, Y1 Resonator_Small

Commit message: restructured the bottom rows
Parts:
- removed MX64-ALPS-4: SPACE LEFT, MX_Alps_Hybrid:MX-2.75U-NoLED, symbol MX_Alps_Hybrid:MX-NoLED
- removed MX65-2: RETURN, MX_Alps_Hybrid:MX-1.5U-NoLED, symbol MX_Alps_Hybrid:MX-NoLED
- removed MX66-ALPS-4: SPACE RIGHT, MX_Alps_Hybrid:MX-2.75U-NoLED, symbol MX_Alps_Hybrid:MX-NoLED
- added D67, D68: D_Small, Diode_SMD:D_0805_2012Metric, symbol Device:D_Small
- added MX61-3: FN, MX_Alps_Hybrid:MX-1U-NoLED, symbol MX_Alps_Hybrid:MX-NoLED
- added MX62-3: CONTROL, MX_Alps_Hybrid:MX-1U-NoLED, symbol MX_Alps_Hybrid:MX-NoLED
- added MX63-3: OPTION, MX_Alps_Hybrid:MX-1U-NoLED, symbol MX_Alps_Hybrid:MX-NoLED
- added MX64-3, MX65-4, MX71-4: CMD, MX_Alps_Hybrid:MX-1U-NoLED, symbol MX_Alps_Hybrid:MX-NoLED
- added MX65-3: LEFT SPACE, MX_Alps_Hybrid:MX-2.75U-ReversedStabilizers-NoLED, symbol MX_Alps_Hybrid:MX-NoLED
- added MX65-5, MX71-5: CMD, MX_Alps_Hybrid:MX-1.25U-NoLED, symbol MX_Alps_Hybrid:MX-NoLED
- added MX66-4: LEFT SPACE, MX_Alps_Hybrid:MX-2U-ReversedStabilizers-NoLED, symbol MX_Alps_Hybrid:MX-NoLED
- added MX66-5: LEFT SPACE, MX_Alps_Hybrid:MX-1.25U-NoLED, symbol MX_Alps_Hybrid:MX-NoLED
- added MX67-5: LEFT CENTRE, MX_Alps_Hybrid:MX-1U-NoLED, symbol MX_Alps_Hybrid:MX-NoLED
- added MX69-5: RIGHT CENTRE, MX_Alps_Hybrid:MX-1U-NoLED, symbol MX_Alps_Hybrid:MX-NoLED
- added MX70-4: RIGHT SPACE, MX_Alps_Hybrid:MX-2U-ReversedStabilizers-NoLED, symbol MX_Alps_Hybrid:MX-NoLED
- added MX70-5: RIGHT SPACE, MX_Alps_Hybrid:MX-1.25U-NoLED, symbol MX_Alps_Hybrid:MX-NoLED
- added MX71-3: RIGHT SPACE, MX_Alps_Hybrid:MX-2.75U-ReversedStabilizers-NoLED, symbol MX_Alps_Hybrid:MX-NoLED
- MX65-1: renamed from MX64-1; value SPACE LEFT -> LEFT SPACE
- MX65-2: renamed from MX64-2; value SPACE LEFT -> LEFT SPACE
- MX71-1: renamed from MX66-1; value SPACE RIGHT -> RIGHT SPACE
- MX71-2: renamed from MX66-2; value SPACE RIGHT -> RIGHT SPACE
- renumbered MX65 to MX68, MX65-1 to MX68-1, MX72-4 to MX72-3, MX69 to MX73, MX69-1 to MX73-1, MX73-4 to MX73-3, MX70 to MX74, MX70-1 to MX74-1, MX74-4 to MX74-3, MX71 to MX75, MX71-1 to MX75-1, MX75-4 to MX75-3
Connections:
- net Col0: now also MX61-3.1 (COL)
- net Col1: now also MX62-3.1 (COL)
- net Col10: now also MX71-1.1 (COL), MX71-2.1 (COL), MX71-3.1 (COL), MX71-4.1 (COL), MX71-5.1 (COL); no longer MX75-1.1 (COL), MX75.1 (COL)
- net Col12: now also MX73-1.1 (COL), MX73.1 (COL)
- net Col13: now also MX74-1.1 (COL), MX74.1 (COL)
- net Col14: now also MX75-1.1 (COL), MX75.1 (COL)
- net Col2: now also MX63-3.1 (COL)
- net Col3: now also MX64-3.1 (COL); no longer MX65-1.1 (COL), MX65-2.1 (COL)
- net Col4: now also MX65-1.1 (COL), MX65-2.1 (COL), MX65-3.1 (COL), MX65-4.1 (COL), MX65-5.1 (COL); no longer MX68-1.1 (COL), MX68.1 (COL)
- net Col5: now also MX66-4.1 (COL), MX66-5.1 (COL); no longer MX71-1.1 (COL), MX71-2.1 (COL)
- net Col6: now also MX67-5.1 (COL)
- net Col7: now also MX68-1.1 (COL), MX68.1 (COL)
- net Col8: now also MX69-5.1 (COL); no longer MX73-1.1 (COL), MX73.1 (COL)
- net Col9: now also MX70-4.1 (COL), MX70-5.1 (COL); no longer MX74-1.1 (COL), MX74.1 (COL)
- net Row4: now also D67.1 (K), D68.1 (K)
- net at MX68-1.2 (ROW), MX68.2 (ROW): now also D68.2 (A); no longer D65.2 (A)
- net at MX65-1.2 (ROW), MX65-2.2 (ROW): now also D65.2 (A), MX65-3.2 (ROW), MX65-4.2 (ROW), MX65-5.2 (ROW); no longer D64.2 (A)
- net at MX75-1.2 (ROW), MX75.2 (ROW): now also D75.2 (A), MX75-3.2 (ROW); no longer D71.2 (A)
- net at MX74-1.2 (ROW), MX74.2 (ROW): now also D74.2 (A), MX74-3.2 (ROW); no longer D70.2 (A)
- net at D61.2 (A), MX61-1.2 (ROW), MX61.2 (ROW): now also MX61-3.2 (ROW)
- net at D62.2 (A), MX62-1.2 (ROW), MX62.2 (ROW): now also MX62-3.2 (ROW)
- net at D63.2 (A), MX63-1.2 (ROW), MX63.2 (ROW): now also MX63-3.2 (ROW)
- net at MX73-1.2 (ROW), MX73.2 (ROW): now also D73.2 (A), MX73-3.2 (ROW); no longer D69.2 (A)
- net at MX71-1.2 (ROW), MX71-2.2 (ROW): now also D71.2 (A), MX71-3.2 (ROW), MX71-4.2 (ROW), MX71-5.2 (ROW); no longer D66.2 (A)
- new net: D64.2 (A), MX64-3.2 (ROW)
- new net: D70.2 (A), MX70-4.2 (ROW), MX70-5.2 (ROW)
- new net: D69.2 (A), MX69-5.2 (ROW)
- new net: D66.2 (A), MX66-4.2 (ROW), MX66-5.2 (ROW)
- new net: D67.2 (A), MX67-5.2 (ROW)
Other:
- moved on the sheet: D61, D62, D63, D64, D65, D66, D69, D70, D71, D72, D73, D74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

Commit message: Traced routes for the new layouts, improved much of the other tracing
Parts:
- MX65-3, MX71-3: footprint MX_Alps_Hybrid:MX-2.75U-ReversedStabilizers-NoLED -> MX_Alps_Hybrid:MX-2.75U-NoLED
Changed lines of the file:
@@
 F 0 "MX71-3" H 15182 8374 60  0000 C CNN
 F 1 "RIGHT SPACE" H 15182 8300 20  0000 C CNN
-F 2 "MX_Alps_Hybrid:MX-2.75U-ReversedStabilizers-NoLED" H 14475 8125 60  0001 C CNN
+F 2 "MX_Alps_Hybrid:MX-2.75U-NoLED" H 14475 8125 60  0001 C CNN
 F 3 "" H 14475 8125 60  0001 C CNN
 	1    15100 8150
@@
 F 0 "MX65-3" H 7682 8374 60  0000 C CNN
 F 1 "LEFT SPACE" H 7682 8300 20  0000 C CNN
-F 2 "MX_Alps_Hybrid:MX-2.75U-ReversedStabilizers-NoLED" H 6975 8125 60  0001 C CNN
+F 2 "MX_Alps_Hybrid:MX-2.75U-NoLED" H 6975 8125 60  0001 C CNN
 F 3 "" H 6975 8125 60  0001 C CNN
 	1    7600 8150
