File: tsuka60.kicad_pcb (KiCad board)
At the start: 2 copper layers, 285 x 95.1 mm, 165 parts, among them SW1 SW_Push, U1 ATmega32U4-AU, Y1 Resonator_Small

Commit message: Started organising bottom rows
Parts:
- removed MX37, MX39, MX52, MX54, MX64, MX65, MX66, MX68: MX-LED, MX_Alps_Hybrid:MX-1U-NoLED
- added D64: D_Small, Diode_SMD:D_0805_2012Metric, B.Cu at (123.2, 537.8)
- added D65: D_Small, Diode_SMD:D_0805_2012Metric, B.Cu at (127.6, 537.8)
- added D70: D_Small, Diode_SMD:D_0805_2012Metric, B.Cu at (123.2, 534.7)
- added D71: D_Small, Diode_SMD:D_0805_2012Metric, B.Cu at (127.6, 534.7)
- added D72: D_Small, Diode_SMD:D_0805_2012Metric, B.Cu at (132.1, 537.8)
- added MX61-1: L-CTRL, MX_Alps_Hybrid:MX-1.25U-NoLED, F.Cu at (107.2, 254.8)
- added MX62-1: L-WIN, MX_Alps_Hybrid:MX-1.25U-NoLED, F.Cu at (131.0, 254.8)
- added MX63-1: L-ALT, MX_Alps_Hybrid:MX-1.25U-NoLED, F.Cu at (154.8, 254.8)
- added MX64-1: BACK SPACE, MX_Alps_Hybrid:MX-2.75U-ReversedStabilizers-NoLED, F.Cu at (192.9, 254.8)
- added MX64-2: BACK SPACE, MX_Alps_Hybrid:MX-3U-ReversedStabilizers-NoLED, F.Cu at (195.3, 292.9)
- added MX65-1: RETURN, MX_Alps_Hybrid:MX-2U-ReversedStabilizers-NoLED, F.Cu at (238.1, 254.8)
- added MX65-2: RETURN, MX_Alps_Hybrid:MX-1.5U-NoLED, F.Cu at (238.1, 292.9)
- added MX67-1: SPACE, MX_Alps_Hybrid:MX-2.75U-ReversedStabilizers-NoLED, F.Cu at (283.4, 254.8)
- added MX67-2: SPACE, MX_Alps_Hybrid:MX-3U-ReversedStabilizers-NoLED, F.Cu at (281.0, 292.9)
- added MX67-3: SPACE, MX_Alps_Hybrid:MX-6.25U-ReversedStabilizers-NoLED, F.Cu at (226.2, 323.1)
- added MX68-3: LEGACY, MX_Alps_Hybrid:MX-1.25U-NoLED, F.Cu at (297.7, 323.1)
- added MX69-1: R-ALT, MX_Alps_Hybrid:MX-1.25U-NoLED, F.Cu at (321.5, 254.8)
- added MX70-1: R-WIN, MX_Alps_Hybrid:MX-1.25U-NoLED, F.Cu at (345.3, 254.8)
- added MX71-1: R-CTRL, MX_Alps_Hybrid:MX-1.25U-NoLED, F.Cu at (369.1, 254.8)
- C1, C2, C3, C4, C5, D1, D10, D11, D12, D13, D14, D15, D16, D17, D18, D19, D2, D20, D21, D22, D23, D24, D25, D26, D27, D28, D29, D3, D30, D31, D32, D33, D34, D35, D36, D37, D38, D39, D4, D40, D41, D42, D43, D44, D45, D46, D47, D48, D49, D5, D50, D51, D52, D53, D54, D55, D56, D57, D58, D59, D6, D60, D61, D62, D63, D64, D65, D66, D67, D68, D69, D7, D70, D71, D72, D73, D74, D75, D8, D9, F1, R1, R2, R3, R4, SW1, U1, USB1, Y1: moved to B.Cu
- MX61: value MX-LED -> L-CTRL; footprint MX_Alps_Hybrid:MX-1U-NoLED -> MX_Alps_Hybrid:MX-1.5U-NoLED
- MX62: value MX-LED -> L-WIN
- MX63: value MX-LED -> L-ALT; footprint MX_Alps_Hybrid:MX-1U-NoLED -> MX_Alps_Hybrid:MX-1.5U-NoLED
- MX67: value MX-LED -> SPACE; footprint MX_Alps_Hybrid:MX-1U-NoLED -> MX_Alps_Hybrid:MX-7U-NoLED
- MX69: value MX-LED -> R-ALT; footprint MX_Alps_Hybrid:MX-1U-NoLED -> MX_Alps_Hybrid:MX-1.5U-NoLED
- MX70: value MX-LED -> R-WIN
- MX71: value MX-LED -> R-CTRL; footprint MX_Alps_Hybrid:MX-1U-NoLED -> MX_Alps_Hybrid:MX-1.5U-NoLED
- MX72: value MX-LED -> LEFT
- MX73: value MX-LED -> DOWN
- MX74: value MX-LED -> UP
- MX75: value MX-LED -> RIGHT
- moved USB1 337.4 mm to (109.5, 101.6)
- moved D26 183.0 mm to (349.1, 513.8)
- moved D18 176.9 mm to (349.1, 510.7)
- moved D4 170.8 mm to (349.1, 507.7)
- moved D2 164.8 mm to (349.1, 504.6)
- moved C5 154.2 mm to (345.3, 499.4)
- moved D13 133.5 mm to (334.6, 489.0)
- moved R1 127.5 mm to (334.6, 486.0)
- moved MX71 111.8 mm to (366.7, 221.5)
- moved MX70 110.2 mm to (342.9, 221.5)
- moved MX69 107.9 mm to (319.1, 221.5)
- moved D12 102.2 mm to (318.9, 473.4)
- moved D14 102.2 mm to (314.4, 473.4)
- moved MX63 100.5 mm to (157.2, 221.5)
- moved MX62 97.0 mm to (133.3, 221.5)
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
Commit message: Start with the layout of diodes
Parts:
- removed D37, D39, D52, D54: D_Small, Diode_SMD:D_0805_2012Metric
- removed the D64 at (130.1, 389.5)
- removed the D64 at (123.2, 537.8)
- removed the D65 at (134.6, 392.6)
- removed the D65 at (127.6, 537.8)
- removed the D70 at (121.2, 392.6)
- removed the D70 at (123.2, 534.7)
- removed the D71 at (116.8, 389.5)
- removed the D71 at (127.6, 534.7)
- removed the D72 at (112.3, 389.5)
- removed the D72 at (132.1, 537.8)
- added D64: D_Small, Diode_SMD:D_0805_2012Metric, B.Cu at (183.4, 65.2)
- added D65: D_Small, Diode_SMD:D_0805_2012Metric, B.Cu at (191.3, 65.2)
- added D70: D_Small, Diode_SMD:D_0805_2012Metric, B.Cu at (231.0, 65.2)
- added D71: D_Small, Diode_SMD:D_0805_2012Metric, B.Cu at (238.9, 65.2)
- added D72: D_Small, Diode_SMD:D_0805_2012Metric, B.Cu at (246.9, 65.2)
- USB1: footprint random-keyboard-parts:Molex-0548190589 -> random-keyboard-parts:Molex-0548190519
- moved Y1 545.4 mm to (478.2, -7.94)
- moved C5 509.5 mm to (495.9, 12.7)
- moved C2 479.3 mm to (481.7, 7.14)
- moved C4 475.0 mm to (476.9, -1.59)
- moved C1 473.5 mm to (488.0, 15.1)
- moved C3 467.0 mm to (475.3, 5.56)
- moved R1 446.6 mm to (121.3, 93.7)
- moved R4 442.7 mm to (477.8, 18.3)
- moved D2 437.9 mm to (128.6, 126.3), turned to 90 degrees
- moved D4 422.7 mm to (166.7, 126.3), turned to 90 degrees
- moved D18 417.2 mm to (147.6, 145.4), turned to 90 degrees
- moved U1 414.9 mm to (497.7, -4.76)
- moved D26 371.6 mm to (300.0, 145.4), turned to 90 degrees
- moved D13 362.7 mm to (338.1, 126.3), turned to 90 degrees
- moved R2 362.3 mm to (107.8, 80.2)
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
Commit message: ready for tracing
Parts:
- removed D66: D_Small, Diode_SMD:D_0805_2012Metric
- MX53: footprint MX_Alps_Hybrid:MX-2U-NoLED -> MX_Alps_Hybrid:MX-2U-ReversedStabilizers-NoLED
- moved U1 292.7 mm to (249.2, 150.0), turned to 270 degrees
- moved C3 278.2 mm to (242.1, 157.2), turned to 180 degrees
- moved R4 276.6 mm to (241.9, 162.7)
- moved C4 276.2 mm to (241.9, 143.7)
- moved C2 272.8 mm to (258.1, 163.5), turned to 180 degrees
- moved C5 266.8 mm to (264.5, 145.3), turned to 180 degrees
- moved Y1 265.7 mm to (264.3, 149.6), turned to 90 degrees
- moved C1 265.3 mm to (251.0, 134.1), turned to 180 degrees
- moved D71 186.4 mm to (374.6, 193.0)
- moved D70 175.2 mm to (350.8, 193.0)
- moved D75 173.8 mm to (377.0, 202.6)
- moved D74 166.7 mm to (358.0, 202.6)
- moved D69 164.8 mm to (327.0, 193.0)
- moved D68 163.2 mm to (303.2, 202.6)
- moved D73 161.3 mm to (338.9, 202.6)
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
Commit message: started tracing
Parts:
- moved D23 0.14 mm to (232.6, 145.4)
- moved D49 0.14 mm to (176.2, 183.5)
- moved D59 0.14 mm to (347.7, 183.5)
Connections:
- MX16 pad 1: Net-(MX16-Pad1) -> Col0
- MX17 pad 1: Net-(MX17-Pad1) -> Col1
- MX18 pad 1: Net-(MX18-Pad1) -> Col2
- MX19 pad 1: Net-(MX19-Pad1) -> Col3
- MX20 pad 1: Net-(MX20-Pad1) -> Col4
- MX21 pad 1: Net-(MX21-Pad1) -> Col5
- MX22 pad 1: Net-(MX22-Pad1) -> Col6
- MX23 pad 1: Net-(MX23-Pad1) -> Col7
- MX24 pad 1: Net-(MX24-Pad1) -> Col8
- MX25 pad 1: Net-(MX25-Pad1) -> Col9
- MX26 pad 1: Net-(MX26-Pad1) -> Col10
- MX27 pad 1: Net-(MX27-Pad1) -> Col11
- MX28 pad 1: Net-(MX28-Pad1) -> Col12
- MX29 pad 1: Net-(MX29-Pad1) -> Col13
- MX30 pad 1: Net-(MX30-Pad1) -> Col14
- MX31 pad 1: Net-(MX31-Pad1) -> Col0
- MX32 pad 1: Net-(MX32-Pad1) -> Col1
- MX33 pad 1: Net-(MX33-Pad1) -> Col2
- MX34 pad 1: Net-(MX34-Pad1) -> Col3
- MX35 pad 1: Net-(MX35-Pad1) -> Col4
- MX36 pad 1: Net-(MX36-Pad1) -> Col5
- MX38 pad 1: Net-(MX38-Pad1) -> Col7
- MX40 pad 1: Net-(MX40-Pad1) -> Col9
- MX41 pad 1: Net-(MX41-Pad1) -> Col10
- MX42 pad 1: Net-(MX42-Pad1) -> Col11
- MX43 pad 1: Net-(MX43-Pad1) -> Col12
- MX44 pad 1: Net-(MX44-Pad1) -> Col13
- MX45 pad 1: Net-(MX45-Pad1) -> Col14
Routing:
- net Net-(D67-Pad2): track 0.00 -> 69.5 mm
- net +5V: track 0.00 -> 57.4 mm
- net Net-(D38-Pad2): track 0.00 -> 18.9 mm
- net Net-(D24-Pad2): track 0.00 -> 16.1 mm
- net D-: track 0.00 -> 16.0 mm
- net Net-(D29-Pad2): track 0.00 -> 15.6 mm
- net Net-(D23-Pad2): track 0.00 -> 12.6 mm
- net Net-(D63-Pad2): track 0.00 -> 10.9 mm
- net Net-(D61-Pad2): track 0.00 -> 10.9 mm
- net Net-(D68-Pad2): track 0.00 -> 10.6 mm
- net Net-(D64-Pad2): track 0.00 -> 10.5 mm
- net Net-(D75-Pad2): track 0.00 -> 10.5 mm
- net Net-(D74-Pad2): track 0.00 -> 10.5 mm
- net Net-(D73-Pad2): track 0.00 -> 10.5 mm
- net Net-(D65-Pad2): track 0.00 -> 10.4 mm
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Other:
- net class Default: trace_width 0.25 -> 0.254
- net class Power added: clearance 0.2, trace_width 0.381, via_dia 0.8, via_drill 0.4

Commit message: tracing
Routing:
- net +5V: track 57.4 -> 218.5 mm
- net Col10: track 0.00 -> 157.9 mm, vias 0 -> 1
- net Col4: track 0.00 -> 129.0 mm
- net Col3: track 0.00 -> 102.5 mm
- net Col11: track 0.00 -> 101.1 mm
- net Col13: track 0.00 -> 100.1 mm
- net Col14: track 0.00 -> 98.8 mm
- net Col12: track 0.00 -> 98.5 mm
- net Col2: track 0.00 -> 84.7 mm
- net Col1: track 0.00 -> 83.2 mm
- net Col6: track 0.00 -> 80.6 mm
- net Col9: track 0.00 -> 64.1 mm
- net Col5: track 0.00 -> 64.1 mm
- net Col0: track 0.00 -> 60.4 mm
- net Col7: track 0.00 -> 37.7 mm
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
Commit message: more traces
Parts:
- moved C5 26.6 mm to (237.9, 146.8), turned to 0 degrees
- moved R1 24.6 mm to (122.2, 127.9), turned to 90 degrees
- moved C2 20.5 mm to (263.1, 143.6)
- moved C3 16.9 mm to (258.0, 162.9), turned to 0 degrees
- moved D17 14.3 mm to (131.0, 145.4)
- moved D29 13.5 mm to (343.7, 145.4)
- moved C4 12.7 mm to (250.6, 134.3), turned to 270 degrees
- moved R3 7.94 mm to (112.7, 127.9)
- moved F1 4.76 mm to (119.1, 127.8)
- moved D40 3.97 mm to (270.7, 164.4)
- moved C1 3.07 mm to (247.9, 134.3), turned to 270 degrees
- moved R2 1.59 mm to (115.9, 127.9)
- moved Y1 0.79 mm to (264.3, 148.8)
- moved D56 0.14 mm to (290.5, 183.5)
- moved D10 0.14 mm to (281.0, 126.3)
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Routing:
- net Row0: track 0.00 -> 309.7 mm, vias 0 -> 2
- net Row3: track 0.00 -> 260.3 mm
- net Row4: track 0.00 -> 245.6 mm
- net Row1: track 0.00 -> 243.6 mm
- net Row2: track 0.00 -> 239.3 mm
- net Col0: track 60.4 -> 221.3 mm
- net Net-(R1-Pad1): track 0.00 -> 159.0 mm, vias 0 -> 2
- net Net-(R3-Pad1): track 0.00 -> 143.7 mm
- net Net-(R2-Pad1): track 0.00 -> 141.3 mm
- net Col1: track 83.2 -> 201.7 mm
- net Col14: track 98.8 -> 206.9 mm
- net Col2: track 84.7 -> 178.6 mm
- net GND: track 9.90 -> 97.7 mm, vias 0 -> 1
- net Col13: track 100.1 -> 183.3 mm
- net Col8: track 18.1 -> 97.6 mm, vias 0 -> 1
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
Commit message: more tracing
Connections:
- U1 pad 31: Col7 -> Col4
- U1 pad 32: Col6 -> Col3
- U1 pad 37: Col4 -> Col7
- U1 pad 38: Col3 -> Col6
Routing:
- net GND: track 97.7 -> 256.3 mm, vias 1 -> 2
- net Col7: track 37.7 -> 151.1 mm, vias 0 -> 2
- net Row1: track 243.6 -> 340.8 mm, vias 0 -> 4
- net Col6: track 80.6 -> 166.6 mm, vias 0 -> 1
- net Col3: track 102.5 -> 168.9 mm
- net Net-(R1-Pad1): track 159.0 -> 204.4 mm, vias 2 -> 4
- net Col10: track 157.0 -> 200.1 mm
- net Col4: track 129.0 -> 170.3 mm, vias 0 -> 1
- net Row2: track 239.3 -> 278.9 mm, vias 0 -> 2
- net Col9: track 138.7 -> 175.1 mm, vias 1 -> 2
- net Col5: track 64.2 -> 100.1 mm
- net +5V: track 268.3 -> 286.6 mm, vias 8 -> 9
- net Net-(R4-Pad2): track 0.00 -> 7.97 mm
- net Net-(D67-Pad2): track 69.5 -> 73.9 mm
- net Col8: track 97.6 -> 93.6 mm
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
Commit message: completed all traces
Connections:
- U1 pad 28: Row3 -> Row4
- U1 pad 29: Row4 -> Row3
- U1 pad 31: Col4 -> Col3
- U1 pad 32: Col3 -> Col4
Routing:
- net Col8: track 93.6 -> 222.4 mm, vias 1 -> 2
- net Row4: track 247.8 -> 298.6 mm, vias 0 -> 2
- net Row3: track 260.3 -> 288.7 mm
- net Col3: track 168.9 -> 195.6 mm, vias 0 -> 2
- net GND: track 256.3 -> 267.4 mm
